Commit message: movebase update

File: husky/husky_description_real/urdf/husky.urdf.xacro (robot description, xacro)
@@ -90,4 +90,10 @@
     <child link="ns0_base_footprint" />
   </joint>
+  <link name="ns0_velodyne"/>
+  <joint name="velodyne_joint" type="fixed">
+    <origin xyz="-0.25 0 0.55" rpy="0 0 0" />
+    <parent link="ns0_base_link" />
+    <child link="ns0_velodyne" />
+  </joint>
   <!-- Inertial link stores the robot's inertial information -->
   <link name="ns0_inertial_link">

File: kimm_robots_description/husky_description/husky_single/husky_panda_rviz_ns0.urdf (robot description, URDF)
Before this commit: robot ns0_husky, 28 links, 27 joints
Links:
- removed link ns0_velodyne
- added link ns0_rviz_velodyne; visual mesh filename=package://velodyne_description/meshes/VLP16_base_1.dae; visual mesh filename=package://velodyne_description/meshes/VLP16_base_2.dae
Joints:
- joint ns0_velodyne_joint: child ns0_velodyne -> ns0_rviz_velodyne

Commit message: update aruco

File: husky/husky_description_real/urdf/husky.urdf.xacro (robot description, xacro)
@@ -96,4 +96,10 @@
     <child link="ns0_velodyne" />
   </joint>
+  <link name="ns0_camera_0"/>
+  <joint name="camera_joint" type="fixed">
+    <origin xyz="0.25 0 0.55" rpy="0 0 0" />
+    <parent link="ns0_base_link" />
+    <child link="ns0_camera_0" />
+  </joint>
   <!-- Inertial link stores the robot's inertial information -->
   <link name="ns0_inertial_link">

Commit message: update qr marker tracking

File: husky/husky_description_real/urdf/husky.urdf.xacro (robot description, xacro)
@@ -96,8 +96,14 @@
     <child link="ns0_velodyne" />
   </joint>
+  <link name="ns0_camera_0_tmp"/>
   <link name="ns0_camera_0"/>
-  <joint name="camera_joint" type="fixed">
-    <origin xyz="0.25 0 0.55" rpy="0 0 0" />
-    <parent link="ns0_base_link" />
+  <joint name="camera_joint0_tmp" type="fixed">
+    <origin xyz="0.40 0 0.3" rpy="0 1.5707 0" />
+    <parent link="ns0_base_link" />
+    <child link="ns0_camera_0_tmp" />
+  </joint>
+  <joint name="camera_joint0" type="fixed">
+    <origin xyz="0 0 0 " rpy="0 0 -1.5707" />
+    <parent link="ns0_camera_0_tmp" />
     <child link="ns0_camera_0" />
   </joint>
