Commit message: update real robot

File: franka_ros/franka_description/robots/panda_arm.urdf.xacro (robot description, xacro)
@@ -1,5 +1,5 @@
 <?xml version='1.0' encoding='utf-8'?>
 <robot xmlns:xacro="http://www.ros.org/wiki/xacro" name="panda">
-  <xacro:arg name="arm_id" default="ns0_panda" /> <!-- Name of this panda -->
+  <xacro:arg name="arm_id" default="ns1_panda" /> <!-- Name of this panda -->
   <xacro:arg name="hand"   default="false" /> <!-- Should a franka_gripper be mounted at the flange?" -->
   <xacro:arg name="gazebo" default="false" /> <!-- Is the robot being simulated in gazebo?" -->

File: franka_ros/franka_description/robots/panda_arm.xacro (robot description, xacro)
@@ -3,5 +3,5 @@
   <!-- safety_distance: Minimum safety distance in [m] by which the collision volumes are expanded and which is enforced during robot motions -->
   <!-- arm_id: Namespace of the panda arm. Serves to differentiate between arms in case of multiple instances. -->
-  <xacro:macro name="panda_arm" params="arm_id:='ns0_panda' description_pkg:='franka_description' connected_to:='' xyz:='0 0 0' rpy:='0 0 0' safety_distance:=0">
+  <xacro:macro name="panda_arm" params="arm_id:='ns1_panda' description_pkg:='franka_description' connected_to:='' xyz:='0 0 0' rpy:='0 0 0' safety_distance:=0">
     <xacro:unless value="${not connected_to}">
       <joint name="${arm_id}_joint_${connected_to}" type="fixed">

File: husky/husky_description_real/urdf/decorations.urdf.xacro (robot description, xacro)
@@ -35,5 +35,5 @@
     <xacro:property name="husky_rear_bumper_extend"  value="$(optenv HUSKY_REAR_BUMPER_EXTEND 0)" />
     <!-- Spawn Husky chassis -->
-    <link name="ns0_top_chassis_link">
+    <link name="ns1_top_chassis_link">
       <visual>
         <origin xyz="0 0 0" rpy="0 0 0" />
@@ -45,10 +45,10 @@
     <!-- Attach chassis to the robot -->
     <joint name="top_chassis_joint" type="fixed">
-      <parent link="ns0_base_link" />
-      <child link="ns0_top_chassis_link" />
+      <parent link="ns1_base_link" />
+      <child link="ns1_top_chassis_link" />
     </joint>
     <xacro:if value="$(optenv HUSKY_USER_RAIL_ENABLED true)">
       <!-- Spawn user rails -->
-      <link name="ns0_user_rail_link">
+      <link name="ns1_user_rail_link">
         <visual>
           <geometry>
@@ -60,11 +60,11 @@
       <joint name="user_rail" type="fixed">
         <origin xyz="0.272 0 0.245" rpy="0 0 0" />
-        <parent link="ns0_base_link" />
-        <child link="ns0_user_rail_link" />
+        <parent link="ns1_base_link" />
+        <child link="ns1_user_rail_link" />
       </joint>
     </xacro:if>
     <!-- Spawn front bumper link -->
     <xacro:if value="${husky_front_bumper_enable}">
-      <link name="ns0_front_bumper_link">
+      <link name="ns1_front_bumper_link">
         <visual>
           <geometry>
@@ -76,9 +76,9 @@
       <joint name="front_bumper" type="fixed">
         <origin xyz="${0.48 + husky_front_bumper_extend} 0 0.091" rpy="0 0 0" />
-        <parent link="ns0_base_link" />
-        <child link="ns0_front_bumper_link" />
+        <parent link="ns1_base_link" />
+        <child link="ns1_front_bumper_link" />
       </joint>
       <xacro:if value="${husky_front_bumper_extend}">
-        <link name="ns0_front_bumper_extension_link">
+        <link name="ns1_front_bumper_extension_link">
             <visual>
                 <geometry>
@@ -89,6 +89,6 @@
         <joint name="front_bumper_extension" type="fixed">
           <origin xyz="${0.48 + husky_front_bumper_extend} 0 0.091" rpy="0 0 0" />
-          <parent link="ns0_base_link" />
-          <child link="ns0_front_bumper_extension_link" />
+          <parent link="ns1_base_link" />
+          <child link="ns1_front_bumper_extension_link" />
         </joint>
       </xacro:if>
@@ -96,5 +96,5 @@
     <!-- Spawn rear bumper link -->
     <xacro:if value="${husky_rear_bumper_enable}">
-      <link name="ns0_rear_bumper_link">
+      <link name="ns1_rear_bumper_link">
         <visual>
           <geometry>
@@ -106,9 +106,9 @@
       <joint name="rear_bumper" type="fixed">
         <origin xyz="${-0.48 - husky_rear_bumper_extend} 0 0.091" rpy="0 0 ${M_PI}" />
-        <parent link="ns0_base_link" />
-        <child link="ns0_rear_bumper_link" />
+        <parent link="ns1_base_link" />
+        <child link="ns1_rear_bumper_link" />
       </joint>
       <xacro:if value="${husky_rear_bumper_extend}">
-        <link name="ns0_rear_bumper_extension_link">
+        <link name="ns1_rear_bumper_extension_link">
             <visual>
                 <geometry>
@@ -119,6 +119,6 @@
         <joint name="rear_bumper_extension" type="fixed">
           <origin xyz="${-0.48 - husky_rear_bumper_extend} 0 0.091" rpy="0 0 ${M_PI}" />
-          <parent link="ns0_base_link" />
-          <child link="ns0_rear_bumper_extension_link" />
+          <parent link="ns1_base_link" />
+          <child link="ns1_rear_bumper_extension_link" />
         </joint>
       </xacro:if>
@@ -127,5 +127,5 @@
       <!-- Spawn the top plate -->
       <xacro:if value="$(optenv HUSKY_LARGE_TOP_PLATE false)">
-        <link name="ns0_top_plate_link">
+        <link name="ns1_top_plate_link">
           <visual>
             <origin xyz="0 0 0" rpy="0 0 0" />
@@ -143,23 +143,23 @@
         <!-- Attach top plate -->
         <joint name="top_plate_joint" type="fixed">
-          <parent link="ns0_base_link" />
-          <child link="ns0_top_plate_link"/>
+          <parent link="ns1_base_link" />
+          <child link="ns1_top_plate_link"/>
           <origin xyz="0.0812 0 0.225" rpy="0 0 0"/>
         </joint>
         <!-- Top plate front link -->
         <joint name="top_plate_front_joint" type="fixed">
-          <parent link="ns0_top_plate_link" />
-          <child link="ns0_top_plate_front_link"/>
+          <parent link="ns1_top_plate_link" />
+          <child link="ns1_top_plate_front_link"/>
           <origin xyz="0.4125 0 0.00672" rpy="0 0 0"/>
         </joint>
         <!-- Top plate rear link-->
         <joint name="top_plate_rear_joint" type="fixed">
-          <parent link="ns0_top_plate_link" />
-          <child link="ns0_top_plate_rear_link"/>
+          <parent link="ns1_top_plate_link" />
+          <child link="ns1_top_plate_rear_link"/>
           <origin xyz="-0.4125 0 0.00672" rpy="0 0 0"/>
         </joint>
       </xacro:if>
       <xacro:unless value="$(optenv HUSKY_LARGE_TOP_PLATE false)">
-        <link name="ns0_top_plate_link">
+        <link name="ns1_top_plate_link">
           <visual>
             <origin xyz="0 0 0" rpy="0 0 0" />
@@ -177,23 +177,23 @@
         <!-- Attach top plate -->
         <joint name="top_plate_joint" type="fixed">
-          <parent link="ns0_base_link" />
-          <child link="ns0_top_plate_link"/>
+          <parent link="ns1_base_link" />
+          <child link="ns1_top_plate_link"/>
           <origin xyz="0.0812 0 0.245" rpy="0 0 0"/>
         </joint>
         <!-- Top plate front link -->
         <joint name="top_plate_front_joint" type="fixed">
-          <parent link="ns0_top_plate_link" />
-          <child link="ns0_top_plate_front_link"/>
+          <parent link="ns1_top_plate_link" />
+          <child link="ns1_top_plate_front_link"/>
           <origin xyz="0.36367 0 0.00639" rpy="0 0 0"/>
         </joint>
         <!-- Top plate rear link-->
         <joint name="top_plate_rear_joint" type="fixed">
-          <parent link="ns0_top_plate_link" />
-          <child link="ns0_top_plate_rear_link"/>
+          <parent link="ns1_top_plate_link" />
+          <child link="ns1_top_plate_rear_link"/>
           <origin xyz="-0.36633 0 0.00639" rpy="0 0 0"/>
         </joint>
       </xacro:unless>
-      <link name="ns0_top_plate_front_link"/>
-      <link name="ns0_top_plate_rear_link"/>
+      <link name="ns1_top_plate_front_link"/>
+      <link name="ns1_top_plate_rear_link"/>
     </xacro:if>
   </xacro:macro>

File: husky/husky_description_real/urdf/husky.urdf.xacro (robot description, xacro)
@@ -63,5 +63,5 @@
   <xacro:property name="wheel_radius" value="0.1651" />
   <!-- Base link is the center of the robot's bottom plate -->
-  <link name="ns0_base_link">
+  <link name="ns1_base_link">
     <visual>
       <origin xyz="0 0 0" rpy="0 0 0" />
@@ -84,30 +84,30 @@
   </link>
   <!-- Base footprint is on the ground under the robot -->
-  <link name="ns0_base_footprint"/>
+  <link name="ns1_base_footprint"/>
   <joint name="base_footprint_joint" type="fixed">
     <origin xyz="0 0 ${wheel_vertical_offset - wheel_radius}" rpy="0 0 0" />
-    <parent link="ns0_base_link" />
-    <child link="ns0_base_footprint" />
-  </joint>
-  <link name="ns0_velodyne"/>
+    <parent link="ns1_base_link" />
+    <child link="ns1_base_footprint" />
+  </joint>
+  <link name="ns1_velodyne"/>
   <joint name="velodyne_joint" type="fixed">
     <origin xyz="-0.25 0 0.55" rpy="0 0 0" />
-    <parent link="ns0_base_link" />
-    <child link="ns0_velodyne" />
-  </joint>
-  <link name="ns0_camera_0_tmp"/>
-  <link name="ns0_camera_0"/>
+    <parent link="ns1_base_link" />
+    <child link="ns1_velodyne" />
+  </joint>
+  <link name="ns1_camera_0_tmp"/>
+  <link name="ns1_camera_0"/>
   <joint name="camera_joint0_tmp" type="fixed">
     <origin xyz="0.40 0 0.3" rpy="0 1.5707 0" />
-    <parent link="ns0_base_link" />
-    <child link="ns0_camera_0_tmp" />
+    <parent link="ns1_base_link" />
+    <child link="ns1_camera_0_tmp" />
   </joint>
   <joint name="camera_joint0" type="fixed">
     <origin xyz="0 0 0 " rpy="0 0 -1.5707" />
-    <parent link="ns0_camera_0_tmp" />
-    <child link="ns0_camera_0" />
+    <parent link="ns1_camera_0_tmp" />
+    <child link="ns1_camera_0" />
   </joint>
   <!-- Inertial link stores the robot's inertial information -->
-  <link name="ns0_inertial_link">
+  <link name="ns1_inertial_link">
     <inertial>
       <mass value="46.034" />
@@ -118,14 +118,14 @@
   <joint name="inertial_joint" type="fixed">
     <origin xyz="0 0 0" rpy="0 0 0" />
-    <parent link="ns0_base_link" />
-    <child link="ns0_inertial_link" />
+    <parent link="ns1_base_link" />
+    <child link="ns1_inertial_link" />
   </joint>
   <!-- IMU Link is the standard mounting position for the UM6 IMU.-->
   <!-- Can be modified with environment variables in /etc/ros/setup.bash -->
-  <link name="ns0_imu_link"/>
+  <link name="ns1_imu_link"/>
   <joint name="imu_joint" type="fixed">
     <origin xyz="$(optenv HUSKY_IMU_XYZ 0.19 0 0.149)" rpy="$(optenv HUSKY_IMU_RPY 0 -1.5708 3.1416)" />
-    <parent link="ns0_base_link" />
-    <child link="ns0_imu_link" />
+    <parent link="ns1_base_link" />
+    <child link="ns1_imu_link" />
   </joint>
   <gazebo reference="imu_link">
@@ -153,6 +153,6 @@
     <joint name="laser_mount_joint" type="fixed">
       <origin xyz="$(arg laser_xyz)" rpy="$(arg laser_rpy)" />
-      <parent link="ns0_top_plate_link" />
-      <child link="ns0_base_laser_mount" />
+      <parent link="ns1_top_plate_link" />
+      <child link="ns1_base_laser_mount" />
     </joint>
   </xacro:if>
@@ -162,6 +162,6 @@
     <joint name="laser_secondary_mount_joint" type="fixed">
       <origin xyz="$(arg laser_secondary_xyz)" rpy="$(arg laser_secondary_rpy)" />
-      <parent link="ns0_top_plate_link" />
-      <child link="ns0_rear_laser_mount" />
+      <parent link="ns1_top_plate_link" />
+      <child link="ns1_rear_laser_mount" />
     </joint>
   </xacro:if>
@@ -180,9 +180,9 @@
   <!-- add the intel realsense to the sensor arch if needed -->
   <xacro:if value="$(arg realsense_enabled)">
-    <link name="ns0_realsense_mountpoint"/>
+    <link name="ns1_realsense_mountpoint"/>
     <joint name="realsense_mountpoint_joint" type="fixed">
       <origin xyz="$(arg realsense_xyz)" rpy="$(arg realsense_rpy)" />
-      <parent link="ns0_$(arg realsense_mount)"/>
-      <child link="ns0_realsense_mountpoint" />
+      <parent link="ns1_$(arg realsense_mount)"/>
+      <child link="ns1_realsense_mountpoint" />
     </joint>
     <xacro:intel_realsense_mount prefix="camera" topic="realsense" parent_link="realsense_mountpoint"/>

File: husky/husky_description_real/urdf/wheel.urdf.xacro (robot description, xacro)
@@ -23,5 +23,5 @@
 <robot xmlns:xacro="http://ros.org/wiki/xacro" name="husky_wheel">
 	<xacro:macro name="husky_wheel" params="wheel_prefix *joint_pose">
-		<link name="ns0_${wheel_prefix}_wheel_link">
+		<link name="ns1_${wheel_prefix}_wheel_link">
 			<inertial>
 				<mass value="2.637" />
@@ -50,6 +50,6 @@
 		</gazebo>
 		<joint name="${wheel_prefix}_wheel" type="continuous">
-			<parent link="ns0_base_link"/>
-			<child link="ns0_${wheel_prefix}_wheel_link"/>
+			<parent link="ns1_base_link"/>
+			<child link="ns1_${wheel_prefix}_wheel_link"/>
 			<xacro:insert_block name="joint_pose"/>
 			<axis xyz="0 1 0" rpy="0 0 0" />

File: kimm_robots_description/husky_description/husky_single/husky_panda_rviz_ns1.urdf (robot description, URDF)
Before this commit: robot ns1_husky, 28 links, 27 joints
Links:
- removed link ns1_velodyne
- added link ns1_rviz_velodyne; visual mesh filename=package://velodyne_description/meshes/VLP16_base_1.dae; visual mesh filename=package://velodyne_description/meshes/VLP16_base_2.dae
Joints:
- joint ns1_velodyne_joint: child ns1_velodyne -> ns1_rviz_velodyne
